Commit message: crane_x7_simple.urdf: Restored joint limits

File: crane_x7_simple.urdf (robot description, URDF)
Before this commit: robot robot, 9 links, 8 joints
Joints:
- joint crane_x7_gripper_finger_a_joint: limit (none) -> lower=0.0046 upper=1.62601 effort=4.0 velocity=4.81710873
- joint crane_x7_lower_arm_fixed_part_joint: limit (none) -> lower=-2.77343 upper=2.77343 effort=4.0 velocity=4.81710873
- joint crane_x7_lower_arm_revolute_part_joint: limit (none) -> lower=-1.570795 upper=1.570795 effort=4.0 velocity=4.81710873
- joint crane_x7_shoulder_fixed_part_pan_joint: limit (none) -> lower=-2.97132 upper=2.97132 effort=10.0 velocity=4.81710873
- joint crane_x7_shoulder_revolute_part_tilt_joint: limit (none) -> lower=-1.570795 upper=1.570795 effort=10.0 velocity=4.81710873
- joint crane_x7_upper_arm_revolute_part_rotate_joint: limit (none) -> lower=-2.80718 upper=0.04141 effort=4.0 velocity=4.81710873
- joint crane_x7_upper_arm_revolute_part_twist_joint: limit (none) -> lower=-1.570795 upper=1.570795 effort=4.0 velocity=4.81710873
- joint crane_x7_wrist_joint: limit (none) -> lower=-2.96365 upper=2.97132 effort=4.0 velocity=4.81710873

Commit message: CRANE-X7 URDF: safer limit for lower arm fixed joint so wires don't snag

File: crane_x7_simple.urdf (robot description, URDF)
Before this commit: robot robot, 9 links, 8 joints
Joints:
- joint crane_x7_lower_arm_fixed_part_joint: limit lower=-2.77343 upper=2.77343 effort=4.0 velocity=4.81710873 -> lower=-0.7417649320975901 upper=0.7417649320975901 effort=4.0 velocity=4.81710873
